File: hardware/awesome-guitar-board.sch (KiCad schematic (older format))
At the start: 0 parts

Commit message: changes on sunday
Changed lines of the file:
@@
-EESchema Schematic File Version 2
-LIBS:power
-LIBS:device
-LIBS:switches
-LIBS:relays
-LIBS:motors
-LIBS:transistors
-LIBS:conn
-LIBS:linear
-LIBS:regul
-LIBS:74xx
-LIBS:cmos4000
-LIBS:adc-dac
-LIBS:memory
-LIBS:xilinx
-LIBS:microcontrollers
-LIBS:dsp
-LIBS:microchip
-LIBS:analog_switches
-LIBS:motorola
-LIBS:texas
-LIBS:intel
-LIBS:audio
-LIBS:interface
-LIBS:digital-audio
-LIBS:philips
-LIBS:display
-LIBS:cypress
-LIBS:siliconi
-LIBS:opto
-LIBS:atmel
-LIBS:contrib
-LIBS:valves
-LIBS:open-automation
+EESchema Schematic File Version 4
 LIBS:awesome-guitar-board-cache
-EELAYER 25 0
+EELAYER 26 0
 EELAYER END
 $Descr A4 11693 8268
 encoding utf-8
-Sheet 1 4
+Sheet 1 5
 Title ""
 Date ""
@@
 S 6900 1950 1450 1125
 U 59CD09F1
-F0 "wireless" 60
-F1 "wireless.sch" 60
+F0 "microcontroller" 60
+F1 "microcontroller.sch" 60
+$EndSheet
+$Sheet
+S 2800 3650 1475 1075
+U 5B847ED8
+F0 "aduio codec" 50
+F1 "digital-codec.sch" 50
 $EndSheet
 $EndSCHEMATC

Commit message: started code
Changed lines of the file:
@@
 EESchema Schematic File Version 4
 LIBS:awesome-guitar-board-cache
-EELAYER 26 0
+EELAYER 29 0
 EELAYER END
 $Descr A4 11693 8268
@@
 $EndDescr
 $Sheet
-S 2775 1950 1450 1125
+S 2500 2000 1450 1125
 U 59CD09A4
 F0 "power" 60
 F1 "power.sch" 60
-$EndSheet
-$Sheet
-S 4875 1950 1450 1125
-U 59CD09B5
-F0 "volume-tone" 60
-F1 "volume-tone.sch" 60
+F2 "V_IN" I L 2500 2350 50
+F3 "GUITAR_OUT" I R 3950 2200 50
+F4 "V_BAT" I L 2500 2250 50
+F5 "V_USB" I L 2500 2150 50
+F6 "3V3" O L 2500 2450 50
 $EndSheet
 $Sheet
@@
 S 2800 3650 1475 1075
 U 5B847ED8
-F0 "aduio codec" 50
+F0 "audio codec" 50
 F1 "digital-codec.sch" 50
 $EndSheet
+$Sheet
+S 5250 1600 1000 850
+U 5C309D83
+F0 "volume-tone" 50
+F1 "volume-tone.sch" 50
+F2 "NECK_OUT" I R 6250 2000 50
+F3 "BRIDGE_OUT" I R 6250 2100 50
+F4 "NECK_IN" I L 5250 1700 50
+F5 "BRIDGE_IN" I L 5250 1800 50
+$EndSheet
 $EndSCHEMATC
