File: hardware/volume-tone.sch (KiCad schematic (older format))
At the start: 6 parts

Commit message: changes on sunday
Parts:
- removed C? (x2): C_0.033uF, Capacitors_SMD:C_0603_HandSoldering, symbol C_0.033uF
- removed RV?: BRIDGE_VOLUME, open-automation:ROT-POT-P160, symbol POT_TRIM-P160KNP-0QC20B500K
- removed RV?: BRIDGE_TONE, open-automation:ROT-POT-P160, symbol POT_TRIM-P160KNP-0QC20B500K
- removed RV?: NECK_VOLUME, open-automation:ROT-POT-P160, symbol POT_TRIM-P160KNP-0QC20B500K
- removed RV?: NECK_TONE, open-automation:ROT-POT-P160, symbol POT_TRIM-P160KNP-0QC20B500K
- added C? (x2): C_0.033, symbol open-automation:C
- added RV? (x4): R_POT, symbol Device:R_POT
Connections:
- wire segments 16 -> 18
Changed lines of the file:
@@
-EESchema Schematic File Version 2
-LIBS:power
-LIBS:device
-LIBS:switches
-LIBS:relays
-LIBS:motors
-LIBS:transistors
-LIBS:conn
-LIBS:linear
-LIBS:regul
-LIBS:74xx
-LIBS:cmos4000
-LIBS:adc-dac
-LIBS:memory
-LIBS:xilinx
-LIBS:microcontrollers
-LIBS:dsp
-LIBS:microchip
-LIBS:analog_switches
-LIBS:motorola
-LIBS:texas
-LIBS:intel
-LIBS:audio
-LIBS:interface
-LIBS:digital-audio
-LIBS:philips
-LIBS:display
-LIBS:cypress
-LIBS:siliconi
-LIBS:opto
-LIBS:atmel
-LIBS:contrib
-LIBS:valves
-LIBS:open-automation
+EESchema Schematic File Version 4
 LIBS:awesome-guitar-board-cache
-EELAYER 25 0
+EELAYER 26 0
 EELAYER END
 $Descr A4 11693 8268
 encoding utf-8
-Sheet 3 4
+Sheet 3 5
 Title ""
 Date ""
@@
 VOLUME-TONE
 $Comp
-L C_0.033uF C?
-U 1 1 59CDA5B2
-P 4575 3875
-F 0 "C?" H 4600 3975 50  0000 L CNN
-F 1 "C_0.033uF" H 4350 3775 50  0000 L CNN
-F 2 "Capacitors_SMD:C_0603_HandSoldering" H 4675 4175 50  0001 C CNN
-F 3 "https://www.digikey.com/product-detail/en/samsung-electro-mechanics-america-inc/CL10B333KB8SFNC/1276-2042-1-ND/3890128" H 4575 3625 50  0001 C CNN
-F 4 "CL10B333KB8SFNC" H 4700 4075 60  0001 C CNN "Part Number"
-	1    4575 3875
-	1    0    0    -1
-$EndComp
-$Comp
-L GND #PWR?
+L power:GND #PWR?
 U 1 1 59CDABF0
 P 4575 4075
@@
 BRIDGE_IN
 $Comp
-L GND #PWR?
+L power:GND #PWR?
 U 1 1 59CDADE5
 P 4800 3100
@@
 	4800 3100 4750 3100
 Wire Wire Line
-	4300 3100 4450 3100
+	4300 3100 4350 3100
 Text GLabel 4650 2900 2    60   Input ~ 0
 BRIDGE_OUT
@@
 	4600 2900 4600 2950
 $Comp
-L C_0.033uF C?
-U 1 1 59CDBF66
-P 6650 3900
-F 0 "C?" H 6675 4000 50  0000 L CNN
-F 1 "C_0.033uF" H 6425 3800 50  0000 L CNN
-F 2 "Capacitors_SMD:C_0603_HandSoldering" H 6750 4200 50  0001 C CNN
-F 3 "https://www.digikey.com/product-detail/en/samsung-electro-mechanics-america-inc/CL10B333KB8SFNC/1276-2042-1-ND/3890128" H 6650 3650 50  0001 C CNN
-F 4 "CL10B333KB8SFNC" H 6775 4100 60  0001 C CNN "Part Number"
-	1    6650 3900
-	1    0    0    -1
-$EndComp
-$Comp
-L GND #PWR?
+L power:GND #PWR?
 U 1 1 59CDBF73
 P 6650 4100
@@
 NECK_IN
 $Comp
-L GND #PWR?
+L power:GND #PWR?
 U 1 1 59CDBF81
 P 6875 3125
@@
 	6875 3125 6825 3125
 Wire Wire Line
-	6375 3125 6525 3125
+	6375 3125 6425 3125
 Text GLabel 6725 2925 2    60   Input ~ 0
 NECK_OUT
@@
 Wire Wire Line
 	6675 2925 6675 2975
+Wire Wire Line
+	4350 3100 4450 3100
+Wire Wire Line
+	6425 3125 6525 3125
 $Comp
-L POT_TRIM-P160KNP-0QC20B500K RV?
-U 1 1 59CE795F
+L Device:R_POT RV?
+U 1 1 5B8481F8
+P 6650 3550
+F 0 "RV?" H 6580 3504 50  0000 R CNN
+F 1 "R_POT" H 6580 3595 50  0000 R CNN
+F 2 "" H 6650 3550 50  0001 C CNN
+F 3 "~" H 6650 3550 50  0001 C CNN
+	1    6650 3550
+	-1   0    0    1
+$EndComp
+$Comp
+L Device:R_POT RV?
+U 1 1 5B848283
+P 6675 3125
+F 0 "RV?" V 6561 3125 50  0000 C CNN
+F 1 "R_POT" V 6470 3125 50  0000 C CNN
+F 2 "" H 6675 3125 50  0001 C CNN
+F 3 "~" H 6675 3125 50  0001 C CNN
+	1    6675 3125
+	0    -1   -1   0
+$EndComp
+$Comp
+L Device:R_POT RV?
+U 1 1 5B8482FB
 P 4600 3100
-F 0 "RV?" V 4675 3175 50  0000 C CNN
-F 1 "BRIDGE_VOLUME" V 4500 3050 50  0000 C CNN
-F 2 "open-automation:ROT-POT-P160" V 4325 3000 50  0001 C CNN
-F 3 "https://www.digikey.com/product-detail/en/tt-electronics-bi/P160KNP-0EC15A500K/987-1722-ND/5957466" V 4425 3100 50  0001 C CNN
-F 4 "P160KNP-0EC15A500K" V 4525 3200 60  0001 C CNN "Part Number"
+F 0 "RV?" H 4530 3146 50  0000 R CNN
+F 1 "R_POT" V 4530 3055 50  0000 R CNN
+F 2 "" H 4600 3100 50  0001 C CNN
+F 3 "~" H 4600 3100 50  0001 C CNN
 	1    4600 3100
 	0    -1   -1   0
 $EndComp
 $Comp
-L POT_TRIM-P160KNP-0QC20B500K RV?
-U 1 1 59CE7993
+L Device:R_POT RV?
+U 1 1 5B84833E
 P 4575 3525
-F 0 "RV?" H 4675 3600 50  0000 C CNN
-F 1 "BRIDGE_TONE" H 4550 3325 50  0000 C CNN
-F 2 "open-automation:ROT-POT-P160" V 4300 3425 50  0001 C CNN
-F 3 "https://www.digikey.com/product-detail/en/tt-electronics-bi/P160KNP-0EC15A500K/987-1722-ND/5957466" V 4400 3525 50  0001 C CNN
-F 4 "P160KNP-0EC15A500K" V 4500 3625 60  0001 C CNN "Part Number"
+F 0 "RV?" H 4505 3479 50  0000 R CNN
+F 1 "R_POT" H 4505 3570 50  0000 R CNN
+F 2 "" H 4575 3525 50  0001 C CNN
+F 3 "~" H 4575 3525 50  0001 C CNN
 	1    4575 3525
 	-1   0    0    1
 $EndComp
 $Comp
-L POT_TRIM-P160KNP-0QC20B500K RV?
-U 1 1 59CE7D77
-P 6675 3125
-F 0 "RV?" V 6750 3200 50  0000 C CNN
-F 1 "NECK_VOLUME" V 6575 3100 50  0000 C CNN
-F 2 "open-automation:ROT-POT-P160" V 6400 3025 50  0001 C CNN
-F 3 "https://www.digikey.com/product-detail/en/tt-electronics-bi/P160KNP-0EC15A500K/987-1722-ND/5957466" V 6500 3125 50  0001 C CNN
-F 4 "P160KNP-0EC15A500K" V 6600 3225 60  0001 C CNN "Part Number"
-	1    6675 3125
-	0    -1   -1   0
+L open-automation:C C?
+U 1 1 5B848C87
+P 6650 3900
+F 0 "C?" H 6765 3946 50  0000 L CNN
+F 1 "C_0.033" H 6765 3855 50  0000 L CNN
+F 2 "" H 6688 3750 50  0000 C CNN
+F 3 "" H 6650 3900 50  0000 C CNN
+	1    6650 3900
+	1    0    0    -1
 $EndComp
 $Comp
-L POT_TRIM-P160KNP-0QC20B500K RV?
-U 1 1 59CE7DD2
-P 6650 3550
-F 0 "RV?" H 6750 3625 50  0000 C CNN
-F 1 "NECK_TONE" H 6650 3350 50  0000 C CNN
-F 2 "open-automation:ROT-POT-P160" V 6375 3450 50  0001 C CNN
-F 3 "https://www.digikey.com/product-detail/en/tt-electronics-bi/P160KNP-0EC15A500K/987-1722-ND/5957466" V 6475 3550 50  0001 C CNN
-F 4 "P160KNP-0EC15A500K" V 6575 3650 60  0001 C CNN "Part Number"
-	1    6650 3550
-	-1   0    0    1
+L open-automation:C C?
+U 1 1 5B848EB9
+P 4575 3875
+F 0 "C?" H 4690 3921 50  0000 L CNN
+F 1 "C_0.033" H 4690 3830 50  0000 L CNN
+F 2 "" H 4613 3725 50  0000 C CNN
+F 3 "" H 4575 3875 50  0000 C CNN
+	1    4575 3875
+	1    0    0    -1
 $EndComp
 $EndSCHEMATC

Commit message: started code
Parts:
- removed C?: C_0.033, symbol open-automation:C
- removed RV? (x2): R_POT, symbol Device:R_POT
- added C?: C_0.033, symbol awesome-guitar-board-rescue:C-open-automation
- added RV? (x2): R_POT, symbol Device:R_POT
- C?: symbol open-automation:C -> awesome-guitar-board-rescue:C-open-automation
Connections:
- net BRIDGE_IN: now also RV?.1, RV?.2
- net BRIDGE_OUT: now also RV?.2
- net GND: now also C?.2, RV?.3
- new net: C?.1, RV?.1
Other:
- moved on the sheet: C?, RV?
Changed lines of the file:
@@
 EESchema Schematic File Version 4
 LIBS:awesome-guitar-board-cache
-EELAYER 26 0
+EELAYER 29 0
 EELAYER END
 $Descr A4 11693 8268
 encoding utf-8
-Sheet 3 5
+Sheet 5 5
 Title ""
 Date ""
@@
 $Comp
 L power:GND #PWR?
-U 1 1 59CDABF0
-P 4575 4075
-F 0 "#PWR?" H 4575 3825 50  0001 C CNN
-F 1 "GND" V 4625 3925 50  0000 C CNN
-F 2 "" H 4575 4075 50  0000 C CNN
-F 3 "" H 4575 4075 50  0000 C CNN
-	1    4575 4075
+U 1 1 59CDBF73
+P 6750 3850
+AR Path="/59CD09B5/59CDBF73" Ref="#PWR?"  Part="1"
+AR Path="/5C309D83/59CDBF73" Ref="#PWR?"  Part="1"
+F 0 "#PWR?" H 6750 3600 50  0001 C CNN
+F 1 "GND" V 6800 3700 50  0000 C CNN
+F 2 "" H 6750 3850 50  0000 C CNN
+F 3 "" H 6750 3850 50  0000 C CNN
+	1    6750 3850
 	1    0    0    -1
 $EndComp
-Text GLabel 4300 3100 0    60   Input ~ 0
-BRIDGE_IN
+Wire Wire Line
+	6750 3850 6750 3800
+Wire Wire Line
+	6750 3500 6750 3450
 $Comp
-L power:GND #PWR?
-U 1 1 59CDADE5
-P 4800 3100
-F 0 "#PWR?" H 4800 2850 50  0001 C CNN
-F 1 "GND" V 4850 2950 50  0000 C CNN
-F 2 "" H 4800 3100 50  0000 C CNN
-F 3 "" H 4800 3100 50  0000 C CNN
-	1    4800 3100
-	0    -1   -1   0
+L awesome-guitar-board-rescue:C-open-automation C?
+U 1 1 5B848C87
+P 6750 3650
+AR Path="/59CD09B5/5B848C87" Ref="C?"  Part="1"
+AR Path="/5C309D83/5B848C87" Ref="C?"  Part="1"
+F 0 "C?" H 6750 3750 50  0000 L CNN
+F 1 "C_0.033" H 6750 3550 50  0000 L CNN
+F 2 "" H 6788 3500 50  0000 C CNN
+F 3 "" H 6750 3650 50  0000 C CNN
+	1    6750 3650
+	1    0    0    -1
+$EndComp
+$Comp
+L Device:R_POT RV?
+U 1 1 5B8481F8
+P 6750 3300
+AR Path="/59CD09B5/5B8481F8" Ref="RV?"  Part="1"
+AR Path="/5C309D83/5B8481F8" Ref="RV?"  Part="1"
+F 0 "RV?" V 6750 3350 50  0000 R CNN
+F 1 "R_POT" V 6650 3400 50  0000 R CNN
+F 2 "" H 6750 3300 50  0001 C CNN
+F 3 "~" H 6750 3300 50  0001 C CNN
+	1    6750 3300
+	-1   0    0    1
 $EndComp
 Wire Wire Line
-	4800 3100 4750 3100
+	6550 2900 6600 2900
 Wire Wire Line
-	4300 3100 4350 3100
-Text GLabel 4650 2900 2    60   Input ~ 0
-BRIDGE_OUT
+	6600 3300 6600 2900
+Connection ~ 6600 2900
 Wire Wire Line
-	4425 3525 4350 3525
-Wire Wire Line
-	4350 3525 4350 3100
-Connection ~ 4350 3100
-Wire Wire Line
-	4575 4075 4575 4025
-Wire Wire Line
-	4575 3725 4575 3675
-Wire Wire Line
-	4650 2900 4600 2900
-Wire Wire Line
-	4600 2900 4600 2950
-$Comp
-L power:GND #PWR?
-U 1 1 59CDBF73
-P 6650 4100
-F 0 "#PWR?" H 6650 3850 50  0001 C CNN
-F 1 "GND" V 6700 3950 50  0000 C CNN
-F 2 "" H 6650 4100 50  0000 C CNN
-F 3 "" H 6650 4100 50  0000 C CNN
-	1    6650 4100
-	1    0    0    -1
-$EndComp
-Text GLabel 6375 3125 0    60   Input ~ 0
-NECK_IN
+	6600 2900 6650 2900
 $Comp
 L power:GND #PWR?
 U 1 1 59CDBF81
-P 6875 3125
-F 0 "#PWR?" H 6875 2875 50  0001 C CNN
-F 1 "GND" V 6925 2975 50  0000 C CNN
-F 2 "" H 6875 3125 50  0000 C CNN
-F 3 "" H 6875 3125 50  0000 C CNN
-	1    6875 3125
+P 7050 2900
+AR Path="/59CD09B5/59CDBF81" Ref="#PWR?"  Part="1"
+AR Path="/5C309D83/59CDBF81" Ref="#PWR?"  Part="1"
+F 0 "#PWR?" H 7050 2650 50  0001 C CNN
+F 1 "GND" V 7000 2750 50  0000 C CNN
+F 2 "" H 7050 2900 50  0000 C CNN
+F 3 "" H 7050 2900 50  0000 C CNN
+	1    7050 2900
 	0    -1   -1   0
-$EndComp
-Wire Wire Line
-	6875 3125 6825 3125
-Wire Wire Line
-	6375 3125 6425 3125
-Text GLabel 6725 2925 2    60   Input ~ 0
-NECK_OUT
-Wire Wire Line
-	6500 3550 6425 3550
-Wire Wire Line
-	6425 3550 6425 3125
-Connection ~ 6425 3125
-Wire Wire Line
-	6650 4100 6650 4050
-Wire Wire Line
-	6650 3750 6650 3700
-Wire Wire Line
-	6725 2925 6675 2925
-Wire Wire Line
-	6675 2925 6675 2975
-Wire Wire Line
-	4350 3100 4450 3100
-Wire Wire Line
-	6425 3125 6525 3125
-$Comp
-L Device:R_POT RV?
-U 1 1 5B8481F8
-P 6650 3550
-F 0 "RV?" H 6580 3504 50  0000 R CNN
-F 1 "R_POT" H 6580 3595 50  0000 R CNN
-F 2 "" H 6650 3550 50  0001 C CNN
-F 3 "~" H 6650 3550 50  0001 C CNN
-	1    6650 3550
-	-1   0    0    1
 $EndComp
 $Comp
 L Device:R_POT RV?
 U 1 1 5B848283
-P 6675 3125
-F 0 "RV?" V 6561 3125 50  0000 C CNN
-F 1 "R_POT" V 6470 3125 50  0000 C CNN
-F 2 "" H 6675 3125 50  0001 C CNN
-F 3 "~" H 6675 3125 50  0001 C CNN
-	1    6675 3125
+P 6800 2900
+AR Path="/59CD09B5/5B848283" Ref="RV?"  Part="1"
+AR Path="/5C309D83/5B848283" Ref="RV?"  Part="1"
+F 0 "RV?" V 6800 2900 50  0000 C CNN
+F 1 "R_POT" V 6700 2900 50  0000 C CNN
+F 2 "" H 6800 2900 50  0001 C CNN
+F 3 "~" H 6800 2900 50  0001 C CNN
+	1    6800 2900
+	0    -1   -1   0
+$EndComp
+Wire Wire Line
+	6950 2900 7050 2900
+Wire Wire Line
+	6850 2700 6800 2700
+Wire Wire Line
+	6800 2700 6800 2750
+$Comp
+L power:GND #PWR?
+U 1 1 5C303384
+P 4750 3850
+AR Path="/59CD09B5/5C303384" Ref="#PWR?"  Part="1"
+AR Path="/5C309D83/5C303384" Ref="#PWR?"  Part="1"
+F 0 "#PWR?" H 4750 3600 50  0001 C CNN
+F 1 "GND" H 4850 3750 50  0000 C CNN
+F 2 "" H 4750 3850 50  0000 C CNN
+F 3 "" H 4750 3850 50  0000 C CNN
+	1    4750 3850
+	1    0    0    -1
+$EndComp
+Wire Wire Line
+	4750 3850 4750 3800
+Wire Wire Line
+	4750 3500 4750 3450
+$Comp
+L awesome-guitar-board-rescue:C-open-automation C?
+U 1 1 5C303391
+P 4750 3650
+AR Path="/59CD09B5/5C303391" Ref="C?"  Part="1"
+AR Path="/5C309D83/5C303391" Ref="C?"  Part="1"
+F 0 "C?" H 4750 3750 50  0000 L CNN
+F 1 "C_0.033" H 4750 3550 50  0000 L CNN
+F 2 "" H 4788 3500 50  0000 C CNN
+F 3 "" H 4750 3650 50  0000 C CNN
+	1    4750 3650
+	1    0    0    -1
+$EndComp
+$Comp
+L Device:R_POT RV?
+U 1 1 5C30339B
+P 4750 3300
+AR Path="/59CD09B5/5C30339B" Ref="RV?"  Part="1"
+AR Path="/5C309D83/5C30339B" Ref="RV?"  Part="1"
+F 0 "RV?" V 4750 3350 50  0000 R CNN
+F 1 "R_POT" V 4650 3400 50  0000 R CNN
+F 2 "" H 4750 3300 50  0001 C CNN
+F 3 "~" H 4750 3300 50  0001 C CNN
+	1    4750 3300
+	-1   0    0    1
+$EndComp
+Wire Wire Line
+	4550 2900 4600 2900
+Wire Wire Line
+	4600 3300 4600 2900
+Connection ~ 4600 2900
+Wire Wire Line
+	4600 2900 4650 2900
+$Comp
+L power:GND #PWR?
+U 1 1 5C3033AA
+P 5050 2900
+AR Path="/59CD09B5/5C3033AA" Ref="#PWR?"  Part="1"
+AR Path="/5C309D83/5C3033AA" Ref="#PWR?"  Part="1"
+F 0 "#PWR?" H 5050 2650 50  0001 C CNN
+F 1 "GND" V 5000 2750 50  0000 C CNN
+F 2 "" H 5050 2900 50  0000 C CNN
+F 3 "" H 5050 2900 50  0000 C CNN
+	1    5050 2900
 	0    -1   -1   0
 $EndComp
 $Comp
 L Device:R_POT RV?
-U 1 1 5B8482FB
-P 4600 3100
-F 0 "RV?" H 4530 3146 50  0000 R CNN
-F 1 "R_POT" V 4530 3055 50  0000 R CNN
-F 2 "" H 4600 3100 50  0001 C CNN
-F 3 "~" H 4600 3100 50  0001 C CNN
-	1    4600 3100
+U 1 1 5C3033B4
+P 4800 2900
+AR Path="/59CD09B5/5C3033B4" Ref="RV?"  Part="1"
+AR Path="/5C309D83/5C3033B4" Ref="RV?"  Part="1"
+F 0 "RV?" V 4800 2900 50  0000 C CNN
+F 1 "R_POT" V 4700 2900 50  0000 C CNN
+F 2 "" H 4800 2900 50  0001 C CNN
+F 3 "~" H 4800 2900 50  0001 C CNN
+	1    4800 2900
 	0    -1   -1   0
 $EndComp
-$Comp
-L Device:R_POT RV?
-U 1 1 5B84833E
-P 4575 3525
-F 0 "RV?" H 4505 3479 50  0000 R CNN
-F 1 "R_POT" H 4505 3570 50  0000 R CNN
-F 2 "" H 4575 3525 50  0001 C CNN
-F 3 "~" H 4575 3525 50  0001 C CNN
-	1    4575 3525
-	-1   0    0    1
-$EndComp
-$Comp
-L open-automation:C C?
-U 1 1 5B848C87
-P 6650 3900
-F 0 "C?" H 6765 3946 50  0000 L CNN
-F 1 "C_0.033" H 6765 3855 50  0000 L CNN
-F 2 "" H 6688 3750 50  0000 C CNN
-F 3 "" H 6650 3900 50  0000 C CNN
-	1    6650 3900
-	1    0    0    -1
-$EndComp
-$Comp
-L open-automation:C C?
-U 1 1 5B848EB9
-P 4575 3875
-F 0 "C?" H 4690 3921 50  0000 L CNN
-F 1 "C_0.033" H 4690 3830 50  0000 L CNN
-F 2 "" H 4613 3725 50  0000 C CNN
-F 3 "" H 4575 3875 50  0000 C CNN
-	1    4575 3875
-	1    0    0    -1
-$EndComp
+Wire Wire Line
+	4950 2900 5050 2900
+Wire Wire Line
+	4850 2700 4800 2700
+Wire Wire Line
+	4800 2700 4800 2750
+Text HLabel 6850 2700 2    50   Input ~ 0
+NECK_OUT
+Text HLabel 4850 2700 2    50   Input ~ 0
+BRIDGE_OUT
+Text HLabel 6550 2900 0    50   Input ~ 0
+NECK_IN
+Text HLabel 4550 2900 0    50   Input ~ 0
+BRIDGE_IN
 $EndSCHEMATC
