File: hardware/digital-codec.sch (KiCad schematic (older format))
At the start: 1 part

Commit message: update
Parts:
- U?: value MAX98089_0 -> MAX98089
Changed lines of the file:
@@
 L max98089_0:MAX98089_0 U?
 U 1 1 5B8326D9
-P 6000 3275
-F 0 "U?" H 7041 3041 50  0000 L CNN
-F 1 "MAX98089_0" H 7041 2950 50  0000 L CNN
-F 2 "Package_DFN_QFN:QFN-56-1EP_7x7mm_P0.4mm_EP5.7x5.7mm" H 6550 4175 50  0001 C CNN
-F 3 "https://www.digikey.com/product-detail/en/maxim-integrated/MAX98089ETN/MAX98089ETN-ND/2744335" H 6000 4375 50  0001 C CNN
-F 4 "MAX98089ETN+" H 7041 2859 50  0000 L CNN "Part Number"
-	1    6000 3275
+P 6775 -650
+F 0 "U?" H 7816 -884 50  0000 L CNN
+F 1 "MAX98089" H 7816 -975 50  0000 L CNN
+F 2 "Package_DFN_QFN:QFN-56-1EP_7x7mm_P0.4mm_EP5.7x5.7mm" H 7325 250 50  0001 C CNN
+F 3 "https://www.digikey.com/product-detail/en/maxim-integrated/MAX98089ETN/MAX98089ETN-ND/2744335" H 6775 450 50  0001 C CNN
+F 4 "MAX98089ETN+" H 7816 -1066 50  0000 L CNN "Part Number"
+	1    6775 -650
 	1    0    0    -1
 $EndComp

Commit message: append
Parts:
- removed U?: MAX98089, Package_DFN_QFN:QFN-56-1EP_7x7mm_P0.4mm_EP5.7x5.7mm, symbol max98089_0:MAX98089_0
- added C? (x8): C_1uF, Capacitor_SMD:C_0603_1608Metric_Pad0.99x1.00mm_HandSolder, symbol open-automation:C_1uF
- added C?: C_2.2uF, Capacitor_SMD:C_0603_1608Metric_Pad0.99x1.00mm_HandSolder, symbol open-automation:C_2.2uF
- added C? (x2): C_0.1uF, Capacitor_SMD:C_0603_1608Metric_Pad0.99x1.00mm_HandSolder, symbol open-automation:C_0.1uF
- added C?: C_10uF, Capacitor_SMD:C_0603_1608Metric_Pad0.99x1.00mm_HandSolder, symbol open-automation:C_10uF
- added R?: R_10k, Resistor_SMD:R_0603_1608Metric_Pad0.99x1.00mm_HandSolder, symbol open-automation:R_10k
- added U?: MAX98089, Package_DFN_QFN:QFN-56-1EP_7x7mm_P0.4mm_EP5.7x5.7mm, symbol Amplifier_Audio:MAX98089
Connections:
- net labels added: +5V, 3v3, GND, I2S_BCLK, I2S_DATA_IN, I2S_WS, L_AUDIO_CODEC_IN, L_AUDIO_IN, R_AUDIO_CODEC_IN, R_AUDIO_IN, SCL, SDA
- wire segments 0 -> 78

Commit message: started code
Parts:
- added U?: MAX98091, Package_DFN_QFN:QFN-48-1EP_6x6mm_P0.4mm_EP4.3x4.3mm_ThermalVias, symbol open-automation:MAX98091
- C? (x8): symbol open-automation:C_1uF -> awesome-guitar-board-rescue:C_1uF-open-automation
- C?: symbol open-automation:C_2.2uF -> awesome-guitar-board-rescue:C_2.2uF-open-automation
- C? (x2): symbol open-automation:C_0.1uF -> awesome-guitar-board-rescue:C_0.1uF-open-automation
- C?: symbol open-automation:C_10uF -> awesome-guitar-board-rescue:C_10uF-open-automation
- R?: symbol open-automation:R_10k -> awesome-guitar-board-rescue:R_10k-open-automation
- U?: symbol Amplifier_Audio:MAX98089 -> awesome-guitar-board-rescue:MAX98089-Amplifier_Audio
Changed lines of the file:
@@
 EESchema Schematic File Version 4
 LIBS:awesome-guitar-board-cache
-EELAYER 26 0
+EELAYER 29 0
 EELAYER END
 $Descr A4 11693 8268
 encoding utf-8
-Sheet 5 5
+Sheet 4 5
 Title ""
 Date ""
@@
 	5950 4800 5950 4875
 $Comp
-L open-automation:GND #PWR?
+L awesome-guitar-board-rescue:GND-open-automation #PWR?
 U 1 1 5B4DCFCE
 P 5950 4875
@@
 Connection ~ 6150 4200
 $Comp
-L open-automation:GND #PWR?
+L awesome-guitar-board-rescue:GND-open-automation #PWR?
 U 1 1 5B32BE2E
 P 7400 4700
@@
 $EndComp
 $Comp
-L open-automation:C_1uF C?
+L awesome-guitar-board-rescue:C_1uF-open-automation C?
 U 1 1 5B33DF15
 P 6200 2450
@@
 	6350 2450 6350 2550
 $Comp
-L open-automation:GND #PWR?
+L awesome-guitar-board-rescue:GND-open-automation #PWR?
 U 1 1 5B3506D8
 P 6350 2550
@@
 	5950 2225 6050 2225
 $Comp
-L open-automation:C_2.2uF C?
+L awesome-guitar-board-rescue:C_2.2uF-open-automation C?
 U 1 1 5B379721
 P 6200 2225
@@
 	6500 2225 6500 2550
 $Comp
-L open-automation:GND #PWR?
+L awesome-guitar-board-rescue:GND-open-automation #PWR?
 U 1 1 5B383127
 P 6500 2550
@@
 	6250 4925 6250 5050
 $Comp
-L open-automation:C_1uF C?
+L awesome-guitar-board-rescue:C_1uF-open-automation C?
 U 1 1 5B3A070A
 P 6400 5050
@@
 	6850 4350 7175 4350
 $Comp
-L open-automation:C_1uF C?
+L awesome-guitar-board-rescue:C_1uF-open-automation C?
 U 1 1 5B3CA38C
 P 7175 4500
@@
 $EndComp
 $Comp
-L open-automation:C_1uF C?
+L awesome-guitar-board-rescue:C_1uF-open-automation C?
 U 1 1 5B3CA4B2
 P 7400 4500
@@
 	7025 4450 7025 4700
 $Comp
-L open-automation:GND #PWR?
+L awesome-guitar-board-rescue:GND-open-automation #PWR?
 U 1 1 5B3F4549
 P 7175 4700
@@
 $EndComp
 $Comp
-L open-automation:GND #PWR?
+L awesome-guitar-board-rescue:GND-open-automation #PWR?
 U 1 1 5B435564
 P 5025 2400
@@
 $EndComp
 $Comp
-L open-automation:C_0.1uF C?
+L awesome-guitar-board-rescue:C_0.1uF-open-automation C?
 U 1 1 5B441011
 P 5175 2600
@@
 Connection ~ 5350 2600
 $Comp
-L open-automation:GND #PWR?
+L awesome-guitar-board-rescue:GND-open-automation #PWR?
 U 1 1 5B46E7FE
 P 5025 2675
@@
 Connection ~ 5550 2350
 $Comp
-L open-automation:GND #PWR?
+L awesome-guitar-board-rescue:GND-open-automation #PWR?
 U 1 1 5B3FED41
 P 7025 4700
@@
 Connection ~ 6050 2850
 $Comp
-L Amplifier_Audio:MAX98089 U?
+L awesome-guitar-board-rescue:MAX98089-Amplifier_Audio U?
 U 1 1 5B46AEA2
 P 5850 3500
@@
 	5550 4800 5550 5250
 $Comp
-L open-automation:+5V #PWR?
+L awesome-guitar-board-rescue:+5V-open-automation #PWR?
 U 1 1 5B3E6C14
 P 5750 5675
@@
 	5300 5250 5550 5250
 $Comp
-L open-automation:C_1uF C?
+L awesome-guitar-board-rescue:C_1uF-open-automation C?
 U 1 1 5B414A02
 P 5150 5250
@@
 $EndComp
 $Comp
-L open-automation:C_1uF C?
+L awesome-guitar-board-rescue:C_1uF-open-automation C?
 U 1 1 5B420336
 P 5975 5250
@@
 	5000 5250 5000 5325
 $Comp
-L open-automation:GND #PWR?
+L awesome-guitar-board-rescue:GND-open-automation #PWR?
 U 1 1 5B45ADC6
 P 6125 5325
@@
 $EndComp
 $Comp
-L open-automation:GND #PWR?
+L awesome-guitar-board-rescue:GND-open-automation #PWR?
 U 1 1 5B45AE7E
 P 5000 5325
@@
 Connection ~ 5600 5500
 $Comp
-L open-automation:C_10uF C?
+L awesome-guitar-board-rescue:C_10uF-open-automation C?
 U 1 1 5B48C588
 P 5900 5500
@@
 	6050 5500 6050 5575
 $Comp
-L open-automation:GND #PWR?
+L awesome-guitar-board-rescue:GND-open-automation #PWR?
 U 1 1 5B4996F5
 P 6050 5575
@@
 	3925 3800 4000 3800
 $Comp
-L open-automation:C_0.1uF C?
+L awesome-guitar-board-rescue:C_0.1uF-open-automation C?
 U 1 1 5B4C0634
 P 4000 3975
@@
 	4000 4150 4000 4125
 $Comp
-L open-automation:GND #PWR?
+L awesome-guitar-board-rescue:GND-open-automation #PWR?
 U 1 1 5B4DABD9
 P 4000 4150
@@
 	4775 2750 4775 2850
 $Comp
-L open-automation:R_10k R?
+L awesome-guitar-board-rescue:R_10k-open-automation R?
 U 1 1 5B53C323
 P 4775 2600
@@
 	4775 2450 4775 2350
 $Comp
-L open-automation:C_1uF C?
+L awesome-guitar-board-rescue:C_1uF-open-automation C?
 U 1 1 5B5934BC
 P 5175 2350
@@
 	5850 2850 5850 2000
 $Comp
-L open-automation:C_1uF C?
+L awesome-guitar-board-rescue:C_1uF-open-automation C?
 U 1 1 5B5E98B2
 P 6200 2000
@@
 	6675 2000 6675 2550
 $Comp
-L open-automation:GND #PWR?
+L awesome-guitar-board-rescue:GND-open-automation #PWR?
 U 1 1 5B6FB0D8
 P 6675 2550
@@
 Text HLabel 5350 2525 1    60   Input ~ 0
 3v3
+$Comp
+L open-automation:MAX98091 U?
+U 1 1 5C3C0959
+P 1700 3850
+F 0 "U?" H 2550 3050 50  0000 L CNN
+F 1 "MAX98091" V 1700 3650 50  0000 L CNN
+F 2 "Package_DFN_QFN:QFN-48-1EP_6x6mm_P0.4mm_EP4.3x4.3mm_ThermalVias" H 1700 3850 50  0001 C CNN
+F 3 "https://www.digikey.com/product-detail/en/maxim-integrated/MAX98091ETM/MAX98091ETM-ND/5049990" H 1700 3850 50  0001 C CNN
+F 4 "MAX98091ETM+" H 1700 3850 50  0001 C CNN "Part Number"
+	1    1700 3850
+	0    1    1    0
+$EndComp
 $EndSCHEMATC

Commit message: added new audio codec
Parts:
- removed C? (x8): C_1uF, Capacitor_SMD:C_0603_1608Metric_Pad0.99x1.00mm_HandSolder, symbol awesome-guitar-board-rescue:C_1uF-open-automation
- removed C?: C_2.2uF, Capacitor_SMD:C_0603_1608Metric_Pad0.99x1.00mm_HandSolder, symbol awesome-guitar-board-rescue:C_2.2uF-open-automation
- removed C? (x2): C_0.1uF, Capacitor_SMD:C_0603_1608Metric_Pad0.99x1.00mm_HandSolder, symbol awesome-guitar-board-rescue:C_0.1uF-open-automation
- removed C?: C_10uF, Capacitor_SMD:C_0603_1608Metric_Pad0.99x1.00mm_HandSolder, symbol awesome-guitar-board-rescue:C_10uF-open-automation
- removed R?: R_10k, Resistor_SMD:R_0603_1608Metric_Pad0.99x1.00mm_HandSolder, symbol awesome-guitar-board-rescue:R_10k-open-automation
- removed U?: MAX98089, Package_DFN_QFN:QFN-56-1EP_7x7mm_P0.4mm_EP5.7x5.7mm, symbol awesome-guitar-board-rescue:MAX98089-Amplifier_Audio
- added C?: C_2.2uF, Capacitor_SMD:C_0603_1608Metric_Pad0.99x1.00mm_HandSolder, symbol awesome-guitar-board-rescue:C_2.2uF-open-automation
- added C? (x15): C_1uF, Capacitor_SMD:C_0603_1608Metric_Pad0.99x1.00mm_HandSolder, symbol awesome-guitar-board-rescue:C_1uF-open-automation
- added C?: C_0.1uF, Capacitor_SMD:C_0603_1608Metric_Pad0.99x1.00mm_HandSolder, symbol awesome-guitar-board-rescue:C_0.1uF-open-automation
- added C? (x2): C_10uF, Capacitor_SMD:C_0603_1608Metric_Pad0.99x1.00mm_HandSolder, symbol awesome-guitar-board-rescue:C_10uF-open-automation
- U?: symbol open-automation:MAX98091 -> awesome-guitar-board-rescue:MAX98091-open-automation
Connections:
- net GND: now also U?.11 (SPKRGND), U?.19 (SPKLGND), U?.2 (HPGND), U?.31 (AGND), U?.37 (DGND), U?.6 (HPSNS), C?.1, C?.1, C?.1, C?.1, C?.1, C?.1, C?.2, C?.2, C?.2, C?.2, C?.2, C?.2
- net I2S_BCLK: now also U?.42 (BCLK)
- net I2S_DATA_IN: now also U?.40 (SDIN)
- net I2S_WS: now also U?.41 (LRCLK)
- net SCL: now also U?.45 (SCL)
- net SDA: now also U?.46 (SDA)
- net at U?.1 (C1N): now also C?.2
- net LOUTR: now reaches U?.10 (RCVN/LOUTR)
- net SPKRN: now reaches U?.12 (SPKRN)
- net SPKRP: now reaches U?.13 (SPKRP)
- net 3V7: now reaches U?.14 (SPKVDD)
- net 3V7: now also U?.15 (SPKVDD), C?.2, C?.2, C?.2
- net SPKLN: now reaches U?.17 (SPKLN)
- net SPKLP: now reaches U?.18 (SPKLP)
- net at U?.20 (IN2/DMC1): now also C?.1
- net at U?.21 (IN1/DMD1): now also C?.1
- net at U?.23 (IN3): now also C?.1
- net at U?.25 (IN5/MDM2): now also C?.2
- net at U?.26 (IN4): now also C?.2
- net at U?.27 (IN6/MDC2): now also C?.2
- net REF: now reaches U?.29 (REF)
- net REF: now also C?.1
- net CPVSS: now reaches U?.3 (CPVSS)
- net CPVSS: now also C?.1
- net BIAS: now reaches U?.30 (BIAS)
- net BIAS: now also C?.1
- net 1V8: now reaches U?.32 (AVDD)
- net 1V8: now also U?.38 (DVDDIO), U?.47 (HPVDD), C?.1, C?.1, C?.2, C?.2
- net 1V2: now reaches U?.36 (DVDD)
- net 1V2: now also C?.2
- net I2S_DATA_OUT: now reaches U?.39 (SDOUT)
- net CPVDD: now reaches U?.4 (CPVDD)
- net CPVDD: now also C?.1
- net CODEC_INT: now reaches U?.43 (~IRQ)
- net MCLK: now reaches U?.44 (MCLK)
- net at U?.48 (C1P): now also C?.1
- net HPL: now reaches U?.5 (HPL)
- net HPR: now reaches U?.7 (HPR)
- net JACKSNS: now reaches U?.8 (JACKSNS)
- net LOUTL: now reaches U?.9 (RCVP/LOUTL)
- new net IN1: C?.2
- new net IN2: C?.2
- new net IN3: C?.2
- new net IN4: C?.1
- new net IN5: C?.1
- new net IN6: C?.1
Other:
- note added: "AVDD"
- note added: "DVDD"
- note added: "DVDDIO"
- note added: "HPVDD"
- note added: "SPKVDD"
- moved on the sheet: U?
