File: hardware/power.sch (KiCad schematic (older format))
At the start: 19 parts

Commit message: changes on sunday
Parts:
- removed BT?: 18650_Battery_Cell_1043, symbol 18650_Battery_Cell_1043
- removed C? (x2): C_1uF, Capacitors_SMD:C_0603, symbol C_1uF
- removed C?: C_0.1uF, Capacitors_SMD:C_0603, symbol C_0.1uF
- removed C?: C_10uF, Capacitors_SMD:C_0603, symbol C_10uF
- removed D?: LED-GREEN-LTST-C191GKT, LEDs:LED_0603, symbol LED-GREEN-LTST-C191GKT
- removed Q?: PMOS-DMG3413L, TO_SOT_Packages_SMD:SOT-23, symbol PMOS-DMG3413L
- removed Q? (x3): BJT-MMBT3904LT3G, TO_SOT_Packages_SMD:SOT-23_Handsoldering, symbol BJT-MMBT3904LT3G
- removed R?: R_1k, Resistors_SMD:R_0603, symbol R_1k
- removed R? (x3): R_10k, Resistors_SMD:R_0603, symbol R_10k
- removed R?: R_2k, Resistors_SMD:R_0603, symbol R_2k
- removed R? (x2): R_1M, Resistors_SMD:R_0603, symbol R_1M
- removed U?: MCP73831T, TO_SOT_Packages_SMD:SOT-23-5, symbol MCP73831T
- removed U?: AZ1117E, open-automation:SPX1117M3, symbol AZ1117E
- added BT?: 18650_Battery_Cell_1043, symbol open-automation:18650_Battery_Cell_1043
- added C? (x2): C_1uF, Capacitor_SMD:C_0603_1608Metric_Pad0.99x1.00mm_HandSolder, symbol open-automation:C_1uF
- added C?: C_10uF, Capacitor_SMD:C_0603_1608Metric_Pad0.99x1.00mm_HandSolder, symbol open-automation:C_10uF
- added C?: C_0.1uF, Capacitor_SMD:C_0603_1608Metric_Pad0.99x1.00mm_HandSolder, symbol open-automation:C_0.1uF
- added D?: LED-GREEN-LTST-C191GKT, LEDs:LED_0603, symbol open-automation:LED-GREEN-LTST-C191GKT
- added Q?: PMOS-DMG3413L, TO_SOT_Packages_SMD:SOT-23, symbol open-automation:PMOS-DMG3413L
- added Q? (x3): 2N3904, Package_TO_SOT_THT:TO-92_Inline, symbol Transistor_BJT:2N3904
- added R? (x3): R_10k, Resistor_SMD:R_0603_1608Metric_Pad0.99x1.00mm_HandSolder, symbol open-automation:R_10k
- added R?: R_2k, Resistors_SMD:R_0603, symbol open-automation:R_2k
- added R?: R_1k, Resistor_SMD:R_0603_1608Metric_Pad0.99x1.00mm_HandSolder, symbol open-automation:R_1k
- added R_1k? (x2): R_1M, Resistors_SMD:R_0603, symbol open-automation:R_1M
- added U?: AZ1117E, TO_SOT_Packages_SMD:SOT-223, symbol open-automation:AZ1117E
- added U?: MCP73831T, TO_SOT_Packages_SMD:SOT-23-5, symbol open-automation:MCP73831T
Connections:
- wire segments 49 -> 61

Commit message: append
Parts:
- R_1k? (x2): symbol open-automation:R_1M -> awesome-guitar-board-rescue:R_1M-open-automation
Changed lines of the file:
@@
 $EndComp
 $Comp
-L open-automation:R_1M R_1k?
+L awesome-guitar-board-rescue:R_1M-open-automation R_1k?
 U 1 1 5B841CCE
 P 3950 5725
@@
 $EndComp
 $Comp
-L open-automation:R_1M R_1k?
+L awesome-guitar-board-rescue:R_1M-open-automation R_1k?
 U 1 1 5B841D8A
 P 3625 6175

Commit message: started code
Parts:
- removed BT?: 18650_Battery_Cell_1043, symbol open-automation:18650_Battery_Cell_1043
- removed C? (x2): C_1uF, Capacitor_SMD:C_0603_1608Metric_Pad0.99x1.00mm_HandSolder, symbol open-automation:C_1uF
- removed C?: C_10uF, Capacitor_SMD:C_0603_1608Metric_Pad0.99x1.00mm_HandSolder, symbol open-automation:C_10uF
- removed C?: C_0.1uF, Capacitor_SMD:C_0603_1608Metric_Pad0.99x1.00mm_HandSolder, symbol open-automation:C_0.1uF
- removed D?: LED-GREEN-LTST-C191GKT, LEDs:LED_0603, symbol open-automation:LED-GREEN-LTST-C191GKT
- removed Q?: PMOS-DMG3413L, TO_SOT_Packages_SMD:SOT-23, symbol open-automation:PMOS-DMG3413L
- removed Q? (x3): 2N3904, Package_TO_SOT_THT:TO-92_Inline, symbol Transistor_BJT:2N3904
- removed R? (x3): R_10k, Resistor_SMD:R_0603_1608Metric_Pad0.99x1.00mm_HandSolder, symbol open-automation:R_10k
- removed R?: R_2k, Resistors_SMD:R_0603, symbol open-automation:R_2k
- removed R?: R_1k, Resistor_SMD:R_0603_1608Metric_Pad0.99x1.00mm_HandSolder, symbol open-automation:R_1k
- removed R_1k? (x2): R_1M, Resistors_SMD:R_0603, symbol awesome-guitar-board-rescue:R_1M-open-automation
- removed U?: AZ1117E, TO_SOT_Packages_SMD:SOT-223, symbol open-automation:AZ1117E
- removed U?: MCP73831T, TO_SOT_Packages_SMD:SOT-23-5, symbol open-automation:MCP73831T
- added BT?: 18650_Battery_Cell_1043, Battery:BatteryHolder_Keystone_1042_1x18650, symbol awesome-guitar-board-rescue:18650_Battery_Cell_1043-liger-rescue
- added C? (x3): C_1uF, Capacitor_SMD:C_0603_1608Metric_Pad1.05x0.95mm_HandSolder, symbol open-automation:C_1uF
- added C? (x2): C_10uF, Capacitor_SMD:C_0603_1608Metric_Pad0.99x1.00mm_HandSolder, symbol awesome-guitar-board-rescue:C_10uF-open-automation
- added C?: C_0.1uF, Capacitor_SMD:C_0603_1608Metric_Pad0.99x1.00mm_HandSolder, symbol awesome-guitar-board-rescue:C_0.1uF-open-automation
- added D?: D_Schottky-BAT20JFILM, Diode_SMD:D_SOD-323_HandSoldering, symbol awesome-guitar-board-rescue:D_Schottky-BAT20JFILM-liger-rescue
- added D?: LED-0603-G, LED_SMD:LED_0603_1608Metric_Pad1.05x0.95mm_HandSolder, symbol open-automation:LED-0603-G
- added Q?: PMOS-DMG3413L, Package_TO_SOT_SMD:SOT-23, symbol awesome-guitar-board-rescue:PMOS-DMG3413L-liger-rescue
- added Q? (x3): 2N3904, Package_TO_SOT_THT:TO-92_Inline, symbol Transistor_BJT:2N3904
- added R?: R_1k, Resistor_SMD:R_0603_1608Metric_Pad1.05x0.95mm_HandSolder, symbol awesome-guitar-board-rescue:R_1k-liger-rescue
- added R?: R_10k, Resistor_SMD:R_0603_1608Metric_Pad1.05x0.95mm_HandSolder, symbol awesome-guitar-board-rescue:R_10k-liger-rescue
- added R?: R_2k, Resistor_SMD:R_0603_1608Metric_Pad1.05x0.95mm_HandSolder, symbol awesome-guitar-board-rescue:R_2k-liger-rescue
- added R? (x2): R_10k, Resistor_SMD:R_0603_1608Metric_Pad0.99x1.00mm_HandSolder, symbol awesome-guitar-board-rescue:R_10k-open-automation
- added R_1k? (x2): R_1M, Resistors_SMD:R_0603, symbol awesome-guitar-board-rescue:R_1M-open-automation-awesome-guitar-board-rescue
- added U?: MCP73831T, Package_TO_SOT_SMD:SOT-23-5_HandSoldering, symbol awesome-guitar-board-rescue:MCP73831T-liger-rescue
- added U?: AP2112, Package_TO_SOT_SMD:SOT-23-5_HandSoldering, symbol awesome-guitar-board-rescue:AP2112-liger-rescue
Connections:
- net labels added: V_BAT, V_IN
- net labels removed: BATTERY, Power, USB
- wire segments 61 -> 76

Commit message: added new audio codec
Parts:
- C? (x3): symbol open-automation:C_1uF -> awesome-guitar-board-rescue:C_1uF-open-automation
- D?: symbol open-automation:LED-0603-G -> awesome-guitar-board-rescue:LED-0603-G-open-automation
Changed lines of the file:
@@
 V_BAT
 $Comp
-L open-automation:C_1uF C?
+L awesome-guitar-board-rescue:C_1uF-open-automation C?
 U 1 1 5B1EEF77
 P 5175 2675
@@
 $EndComp
 $Comp
-L open-automation:C_1uF C?
+L awesome-guitar-board-rescue:C_1uF-open-automation C?
 U 1 1 5B1EF368
 P 3550 2650
@@
 $EndComp
 $Comp
-L open-automation:C_1uF C?
+L awesome-guitar-board-rescue:C_1uF-open-automation C?
 U 1 1 5B1EF9E4
 P 8750 2700
@@
 $EndComp
 $Comp
-L open-automation:LED-0603-G D?
+L awesome-guitar-board-rescue:LED-0603-G-open-automation D?
 U 1 1 5BBE79A0
 P 6425 2650
